File: PCB/PiicoDev-Raspberry-Pi-Adapter.sch (KiCad schematic (older format))
At the start: 14 parts, among them J1 Raspberry_Pi_2_3, J2 Conn_PiicoDev_socket, J3 Conn_PiicoDev_socket, J4 Conn_PiicoDev_socket, J5 Conn_PiicoDev_socket, J6 Prototyping Header

Commit message: update pdf to v13
Other:
- note added: "Series resistance to damp waveform for long buses.\nLong buses can present destructive undershoot, exceeding absolute-maximum rating of the RPi"
Changed lines of the file:
@@
 $EndDescr
 $Comp
-L power:+3V3 #PWR08
+L power:+3V3 #PWR?
 U 1 1 602A11D2
 P 8300 1600
-F 0 "#PWR08" H 8300 1450 50  0001 C CNN
+F 0 "#PWR?" H 8300 1450 50  0001 C CNN
 F 1 "+3V3" H 8315 1773 50  0000 C CNN
 F 2 "" H 8300 1600 50  0001 C CNN
@@
 $EndComp
 $Comp
-L power:GND #PWR012
+L power:GND #PWR?
 U 1 1 602A1DA4
 P 8400 2100
-F 0 "#PWR012" H 8400 1850 50  0001 C CNN
+F 0 "#PWR?" H 8400 1850 50  0001 C CNN
 F 1 "GND" H 8405 1927 50  0000 C CNN
 F 2 "" H 8400 2100 50  0001 C CNN
@@
 	8650 1800 8700 1800
 $Comp
-L power:+3V3 #PWR09
+L power:+3V3 #PWR?
 U 1 1 602A7B49
 P 8300 2750
-F 0 "#PWR09" H 8300 2600 50  0001 C CNN
+F 0 "#PWR?" H 8300 2600 50  0001 C CNN
 F 1 "+3V3" H 8315 2923 50  0000 C CNN
 F 2 "" H 8300 2750 50  0001 C CNN
@@
 $EndComp
 $Comp
-L power:GND #PWR013
+L power:GND #PWR?
 U 1 1 602A7B4F
 P 8400 3250
-F 0 "#PWR013" H 8400 3000 50  0001 C CNN
+F 0 "#PWR?" H 8400 3000 50  0001 C CNN
 F 1 "GND" H 8405 3077 50  0000 C CNN
 F 2 "" H 8400 3250 50  0001 C CNN
@@
 	8650 2950 8700 2950
 $Comp
-L power:+3V3 #PWR010
+L power:+3V3 #PWR?
 U 1 1 602A891A
 P 8300 3850
-F 0 "#PWR010" H 8300 3700 50  0001 C CNN
+F 0 "#PWR?" H 8300 3700 50  0001 C CNN
 F 1 "+3V3" H 8315 4023 50  0000 C CNN
 F 2 "" H 8300 3850 50  0001 C CNN
@@
 $EndComp
 $Comp
-L power:GND #PWR014
+L power:GND #PWR?
 U 1 1 602A8920
 P 8400 4350
-F 0 "#PWR014" H 8400 4100 50  0001 C CNN
+F 0 "#PWR?" H 8400 4100 50  0001 C CNN
 F 1 "GND" H 8405 4177 50  0000 C CNN
 F 2 "" H 8400 4350 50  0001 C CNN
@@
 	8650 4050 8700 4050
 $Comp
-L power:+3V3 #PWR011
+L power:+3V3 #PWR?
 U 1 1 602AA2FA
 P 8300 5000
-F 0 "#PWR011" H 8300 4850 50  0001 C CNN
+F 0 "#PWR?" H 8300 4850 50  0001 C CNN
 F 1 "+3V3" H 8315 5173 50  0000 C CNN
 F 2 "" H 8300 5000 50  0001 C CNN
@@
 $EndComp
 $Comp
-L power:GND #PWR015
+L power:GND #PWR?
 U 1 1 602AA300
 P 8400 5500
-F 0 "#PWR015" H 8400 5250 50  0001 C CNN
+F 0 "#PWR?" H 8400 5250 50  0001 C CNN
 F 1 "GND" H 8405 5327 50  0000 C CNN
 F 2 "" H 8400 5500 50  0001 C CNN
@@
 $EndComp
 $Comp
-L power:GND #PWR01
+L power:GND #PWR?
 U 1 1 602B532C
 P 2150 5250
-F 0 "#PWR01" H 2150 5000 50  0001 C CNN
+F 0 "#PWR?" H 2150 5000 50  0001 C CNN
 F 1 "GND" H 2155 5077 50  0000 C CNN
 F 2 "" H 2150 5250 50  0001 C CNN
@@
 SCL
 $Comp
-L power:+3V3 #PWR03
+L power:+3V3 #PWR?
 U 1 1 602B762E
 P 2650 2400
-F 0 "#PWR03" H 2650 2250 50  0001 C CNN
+F 0 "#PWR?" H 2650 2250 50  0001 C CNN
 F 1 "+3V3" H 2665 2573 50  0000 C CNN
 F 2 "" H 2650 2400 50  0001 C CNN
@@
 $EndComp
 $Comp
-L power:+3V3 #PWR05
+L power:+3V3 #PWR?
 U 1 1 602C7AEC
 P 5350 3150
-F 0 "#PWR05" H 5350 3000 50  0001 C CNN
+F 0 "#PWR?" H 5350 3000 50  0001 C CNN
 F 1 "+3V3" H 5365 3323 50  0000 C CNN
 F 2 "" H 5350 3150 50  0001 C CNN
@@
 	5350 3150 5800 3150
 $Comp
-L power:+5V #PWR02
+L power:+5V #PWR?
 U 1 1 602C8A49
 P 2350 2400
-F 0 "#PWR02" H 2350 2250 50  0001 C CNN
+F 0 "#PWR?" H 2350 2250 50  0001 C CNN
 F 1 "+5V" H 2365 2573 50  0000 C CNN
 F 2 "" H 2350 2400 50  0001 C CNN
@@
 	2650 2450 2650 2400
 $Comp
-L power:+5V #PWR07
+L power:+5V #PWR?
 U 1 1 602CAD3B
 P 5600 3050
-F 0 "#PWR07" H 5600 2900 50  0001 C CNN
+F 0 "#PWR?" H 5600 2900 50  0001 C CNN
 F 1 "+5V" H 5615 3223 50  0000 C CNN
 F 2 "" H 5600 3050 50  0001 C CNN
@@
 	5600 3050 5800 3050
 $Comp
-L power:GND #PWR06
+L power:GND #PWR?
 U 1 1 602CC0E8
 P 5350 3350
-F 0 "#PWR06" H 5350 3100 50  0001 C CNN
+F 0 "#PWR?" H 5350 3100 50  0001 C CNN
 F 1 "GND" H 5355 3177 50  0000 C CNN
 F 2 "" H 5350 3350 50  0001 C CNN
@@
 $EndComp
 $Comp
-L power:+3V3 #PWR04
+L power:+3V3 #PWR?
 U 1 1 6045CC2C
 P 4450 6250
-F 0 "#PWR04" H 4450 6100 50  0001 C CNN
+F 0 "#PWR?" H 4450 6100 50  0001 C CNN
 F 1 "+3V3" H 4465 6423 50  0000 C CNN
 F 2 "" H 4450 6250 50  0001 C CNN
@@
 	8400 3850 8700 3850
 $Comp
-L power:PWR_FLAG #FLG0101
+L power:PWR_FLAG #FLG?
 U 1 1 61E658F6
 P 5650 6900
-F 0 "#FLG0101" H 5650 6975 50  0001 C CNN
+F 0 "#FLG?" H 5650 6975 50  0001 C CNN
 F 1 "PWR_FLAG" H 5650 7073 50  0000 C CNN
 F 2 "" H 5650 6900 50  0001 C CNN
@@
 $EndComp
 $Comp
-L power:GND #PWR0101
+L power:GND #PWR?
 U 1 1 61E65F24
 P 5650 7000
-F 0 "#PWR0101" H 5650 6750 50  0001 C CNN
+F 0 "#PWR?" H 5650 6750 50  0001 C CNN
 F 1 "GND" H 5655 6827 50  0000 C CNN
 F 2 "" H 5650 7000 50  0001 C CNN
@@
 	5650 6900 5650 7000
 $Comp
-L power:PWR_FLAG #FLG0102
+L power:PWR_FLAG #FLG?
 U 1 1 61E699BD
 P 6100 7000
-F 0 "#FLG0102" H 6100 7075 50  0001 C CNN
+F 0 "#FLG?" H 6100 7075 50  0001 C CNN
 F 1 "PWR_FLAG" H 6100 7173 50  0000 C CNN
 F 2 "" H 6100 7000 50  0001 C CNN
@@
 $EndComp
 $Comp
-L power:+3V3 #PWR0102
+L power:+3V3 #PWR?
 U 1 1 61E6AB9F
 P 6100 6900
-F 0 "#PWR0102" H 6100 6750 50  0001 C CNN
+F 0 "#PWR?" H 6100 6750 50  0001 C CNN
 F 1 "+3V3" H 6115 7073 50  0000 C CNN
 F 2 "" H 6100 6900 50  0001 C CNN
@@
 ERC Config
 $Comp
-L power:PWR_FLAG #FLG0103
+L power:PWR_FLAG #FLG?
 U 1 1 61E743DE
 P 6550 7000
-F 0 "#FLG0103" H 6550 7075 50  0001 C CNN
+F 0 "#FLG?" H 6550 7075 50  0001 C CNN
 F 1 "PWR_FLAG" H 6550 7173 50  0000 C CNN
 F 2 "" H 6550 7000 50  0001 C CNN
@@
 $EndComp
 $Comp
-L power:+5V #PWR0103
+L power:+5V #PWR?
 U 1 1 61E74F8E
 P 6550 6900
-F 0 "#PWR0103" H 6550 6750 50  0001 C CNN
+F 0 "#PWR?" H 6550 6750 50  0001 C CNN
 F 1 "+5V" H 6565 7073 50  0000 C CNN
 F 2 "" H 6550 6900 50  0001 C CNN
@@
 Wire Wire Line
 	8400 5000 8400 5500
+Text Notes 3950 1700 0    50   ~ 0
+Series resistance to damp waveform for long buses.\nLong buses can present destructive undershoot, exceeding absolute-maximum rating of the RPi
+Wire Notes Line style solid
+	3950 3000 3950 1750
+Wire Notes Line style solid
+	3950 1750 7650 1750
 $EndSCHEMATC
